Commit message: fix(arm): align URDF and gripper model with raw 96..4000 limits

File: catkin_ws/src/actuator/arm/urdf/arm.urdf (robot description, URDF)
Before this commit: robot arm, 7 links, 6 joints
Joints:
- joint joint1: limit lower=-2.3562 upper=2.3562 effort=0 velocity=0 -> lower=-2.7593024632132037 upper=2.7820127715524072 effort=0 velocity=0
- joint joint2: limit lower=-1.5708 upper=1.5708 effort=0 velocity=0 -> lower=-2.7189056420158937 upper=2.855993321445266 effort=0 velocity=0
- joint joint3: limit lower=-1.5708 upper=1.5708 effort=0 velocity=0 -> lower=-2.855993321445266 upper=2.7189056420158937 effort=0 velocity=0
- joint joint4: limit lower=-1.5708 upper=1.5708 effort=0 velocity=0 -> lower=-2.855993321445266 upper=2.7189056420158937 effort=0 velocity=0
- joint joint5: limit lower=-2.3562 upper=2.3562 effort=0 velocity=0 -> lower=-2.7593024632132037 upper=2.7820127715524072 effort=0 velocity=0
- joint joint6: limit lower=0 upper=0 effort=0 velocity=0 -> lower=-1.2851969946503699 upper=4.289701968810791 effort=0 velocity=0
